File: lab4p1/lab4p1.kicad_sch (KiCad schematic)
At the start: 6 parts, among them J1 9V, SW1 SW_SPDT

Commit message: PCB design pics
Parts:
- C1: footprint (none) -> Capacitor_THT:CP_Radial_Tantal_D5.0mm_P5.00mm
- D1: footprint (none) -> LED_THT:LED_D5.0mm
- J1: footprint (none) -> Connector_JST:JST_PH_B2B-PH-K_1x02_P2.00mm_Vertical
- R1, R2: footprint (none) -> Resistor_THT:R_Axial_DIN0516_L15.5mm_D5.0mm_P20.32mm_Horizontal
- SW1: footprint (none) -> Button_Switch_THT:SW_E-Switch_EG1224_SPDT_Angled
Changed lines of the file:
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@@
+    (stroke (width 0) (type default) (color 0 0 0 0))
+  )
+  (wire (pts (xy 120.65 33.02) (xy 121.92 33.02))
     (stroke (width 0) (type default) (color 0 0 0 0))
   )
@@
       (effects (font (size 1.27 1.27)) (justify right))
     )
-    (property "Footprint" "" (id 2) (at 91.44 53.34 0)
-      (effects (font (size 1.27 1.27)) hide)
-    )
+    (property "Footprint" "Connector_JST:JST_PH_B2B-PH-K_1x02_P2.00mm_Vertical" (id 2) (at 91.44 53.34 0))
     (property "Datasheet" "~" (id 3) (at 91.44 53.34 0)
       (effects (font (size 1.27 1.27)) hide)
@@
       (effects (font (size 1.27 1.27)) (justify left))
     )
-    (property "Footprint" "" (id 2) (at 122.8852 52.07 0)
-      (effects (font (size 1.27 1.27)) hide)
-    )
+    (property "Footprint" "Capacitor_THT:CP_Radial_Tantal_D5.0mm_P5.00mm" (id 2) (at 122.8852 52.07 0))
     (property "Datasheet" "~" (id 3) (at 121.92 48.26 0)
       (effects (font (size 1.27 1.27)) hide)
@@
     (property "Reference" "R2" (id 0) (at 104.14 29.21 90))
     (property "Value" "2.2 kΩ" (id 1) (at 104.14 31.75 90))
-    (property "Footprint" "" (id 2) (at 104.14 37.338 90)
-      (effects (font (size 1.27 1.27)) hide)
-    )
+    (property "Footprint" "Resistor_THT:R_Axial_DIN0516_L15.5mm_D5.0mm_P20.32mm_Horizontal" (id 2) (at 104.14 37.338 90))
     (property "Datasheet" "~" (id 3) (at 104.14 35.56 0)
       (effects (font (size 1.27 1.27)) hide)
@@
     (property "Reference" "SW1" (id 0) (at 115.57 27.94 0))
     (property "Value" "SW_SPDT" (id 1) (at 115.57 30.48 0))
-    (property "Footprint" "" (id 2) (at 115.57 35.56 0)
-      (effects (font (size 1.27 1.27)) hide)
-    )
+    (property "Footprint" "Button_Switch_THT:SW_E-Switch_EG1224_SPDT_Angled" (id 2) (at 115.57 35.56 0))
     (property "Datasheet" "~" (id 3) (at 115.57 35.56 0)
       (effects (font (size 1.27 1.27)) hide)
@@
       (effects (font (size 1.27 1.27)) (justify right))
     )
-    (property "Footprint" "" (id 2) (at 143.51 60.96 0)
-      (effects (font (size 1.27 1.27)) hide)
-    )
+    (property "Footprint" "LED_THT:LED_D5.0mm" (id 2) (at 143.51 60.96 0))
     (property "Datasheet" "~" (id 3) (at 143.51 60.96 0)
       (effects (font (size 1.27 1.27)) hide)
@@
       (effects (font (size 1.27 1.27)) (justify left))
     )
-    (property "Footprint" "" (id 2) (at 141.732 46.99 90)
-      (effects (font (size 1.27 1.27)) hide)
-    )
+    (property "Footprint" "Resistor_THT:R_Axial_DIN0516_L15.5mm_D5.0mm_P20.32mm_Horizontal" (id 2) (at 141.732 46.99 90))
     (property "Datasheet" "~" (id 3) (at 143.51 46.99 0)
       (effects (font (size 1.27 1.27)) hide)
@@
   (symbol_instances
     (path "/6b469276-f5c0-4aa3-8cda-f87973d71757"
-      (reference "C1") (unit 1) (value "4.7μF") (footprint "")
+      (reference "C1") (unit 1) (value "4.7μF") (footprint "Capacitor_THT:CP_Radial_Tantal_D5.0mm_P5.00mm")
     )
     (path "/f09ec940-8b5e-44e3-bf17-f511fdec4964"
-      (reference "D1") (unit 1) (value "LED") (footprint "")
+      (reference "D1") (unit 1) (value "LED") (footprint "LED_THT:LED_D5.0mm")
     )
     (path "/34de9b4d-5453-48ce-965b-f253c42dc050"
-      (reference "J1") (unit 1) (value "9V") (footprint "")
+      (reference "J1") (unit 1) (value "9V") (footprint "Connector_JST:JST_PH_B2B-PH-K_1x02_P2.00mm_Vertical")
     )
     (path "/facd4255-fe5c-4a3c-8ea0-06fa8b801dea"
-      (reference "R1") (unit 1) (value "20 kΩ") (footprint "")
+      (reference "R1") (unit 1) (value "20 kΩ") (footprint "Resistor_THT:R_Axial_DIN0516_L15.5mm_D5.0mm_P20.32mm_Horizontal")
     )
     (path "/8d4f9912-6fb6-408f-917c-929df67c5436"
-      (reference "R2") (unit 1) (value "2.2 kΩ") (footprint "")
+      (reference "R2") (unit 1) (value "2.2 kΩ") (footprint "Resistor_THT:R_Axial_DIN0516_L15.5mm_D5.0mm_P20.32mm_Horizontal")
     )
     (path "/a629cdf2-ea52-434a-92b9-2622decbad84"
-      (reference "SW1") (unit 1) (value "SW_SPDT") (footprint "")
+      (reference "SW1") (unit 1) (value "SW_SPDT") (footprint "Button_Switch_THT:SW_E-Switch_EG1224_SPDT_Angled")
     )
   )
